Commit message: coloring

File: urdf/demo.urdf (robot description, URDF)
Before this commit: robot magician, 5 links, 4 joints
Links:
- added link link_7; collision mesh filename=package://magician/meshes/link_7.STL; visual mesh filename=package://magician/meshes/link_7.STL
- link link_1: geometry collision mesh filename=package://magician/meshes/link_1.STL; visual mesh filename=package://magician/meshes/link_1.dae
- link link_2: geometry collision mesh filename=package://magician/meshes/link_2.STL; visual mesh filename=package://magician/meshes/link_2.dae
- link link_5: geometry collision mesh filename=package://magician/meshes/link_5.dae; visual mesh filename=package://magician/meshes/link_5.dae
Joints:
- added joint joint_7: type revolute, parent link_6, child link_7, origin xyz=0 0 0 rpy=0 3.14159265 0, axis 0 0 1, limit lower=-3.14159265 upper=3.14159265 effort=150.0 velocity=3.15

Commit message: edit the urdf

File: urdf/demo.urdf (robot description, URDF)
Before this commit: robot magician, 6 links, 5 joints
Joints:
- joint joint_7: origin xyz=0 0 0 rpy=0 3.14159265 0 -> xyz=-0.0328 0.02871 0 rpy=0 3.14159265 0
